Commit message: release: dual-arch (x86_64 + aarch64) 20260525_095000

File: src/human_data/urdf/nexus-arm-v15-right.urdf (robot description, URDF)
Before this commit: robot nexus-arm-v15-right, 9 links, 8 joints
Joints:
- joint gripper_Joint: limit lower=-0.35 upper=0 effort=0.8 velocity=15.708 -> lower=-0.628 upper=0 effort=0.8 velocity=15.708

Commit message: release: dual-arch (x86_64 + aarch64) 20260527_154315

File: src/human_data/urdf/nexus-arm-v15-right.urdf (robot description, URDF)
Before this commit: robot nexus-arm-v15-right, 9 links, 8 joints
Links:
- link base_link: mass 1.33721444594961 -> 1.33721444591793
- link gripper_Link: mass 0.0203179842649809 -> 0.0203179850333118
- link link2_Link: mass 0.817693429930293 -> 0.817693429898626
- link link3_Link: mass 1.75399504489588 -> 0.271751634815028
- link link4_Link: mass 0.283402486350328 -> 0.283402825354015
- link link5_Link: mass 0.313095244504967 -> 0.313095250711416
- link link6_Link: mass 0.346703008063088 -> 0.346716592638755
Joints:
- joint gripper_Joint: limit lower=-0.628 upper=0 effort=0.8 velocity=15.708 -> lower=-0.63 upper=0 effort=0.8 velocity=15.708; origin xyz=0.032764 0.17274 0.0177 rpy=0 0 -1.5708 -> xyz=0.032764 0.16888 -0.031841 rpy=0 0 0
- joint link1_Joint: axis 0 0 -1 -> 0 0 1
- joint link2_Joint: origin xyz=-2.3691E-05 -0.014493 0.06 rpy=0 0 0 -> xyz=-2.36911467972752E-05 -0.0144929879654747 0.06 rpy=0 0 0
- joint link3_Joint: origin xyz=0 0.00425 0.11 rpy=0 0 0 -> xyz=0 0.00424999999999998 0.109999318004603 rpy=0 0 0
- joint link4_Joint: origin xyz=-0.10999 0.01025 0 rpy=0 0 0 -> xyz=-0.109992581095629 0.0102500000277369 0 rpy=0 0 0

File: src/robot_controller/urdf/nexus-arm-v15-right.urdf (robot description, URDF)
Before this commit: robot nexus-arm-v15-right, 9 links, 8 joints
Links:
- link base_link: mass 1.33721444594961 -> 1.33721444591793
- link gripper_Link: mass 0.0203179842649809 -> 0.0203179850333118
- link link2_Link: mass 0.817693429930293 -> 0.817693429898626
- link link3_Link: mass 1.75399504489588 -> 0.271751634815028
- link link4_Link: mass 0.283402486350328 -> 0.283402825354015
- link link5_Link: mass 0.313095244504967 -> 0.313095250711416
- link link6_Link: mass 0.346703008063088 -> 0.346716592638755
Joints:
- joint gripper_Joint: limit lower=-0.35 upper=0 effort=0.8 velocity=15.708 -> lower=-0.63 upper=0 effort=0.8 velocity=15.708; origin xyz=0.032764 0.17274 0.0177 rpy=0 0 -1.5708 -> xyz=0.032764 0.16888 -0.031841 rpy=0 0 0
- joint link1_Joint: axis 0 0 -1 -> 0 0 1
- joint link2_Joint: origin xyz=-2.3691E-05 -0.014493 0.06 rpy=0 0 0 -> xyz=-2.36911467972752E-05 -0.0144929879654747 0.06 rpy=0 0 0
- joint link3_Joint: origin xyz=0 0.00425 0.11 rpy=0 0 0 -> xyz=0 0.00424999999999998 0.109999318004603 rpy=0 0 0
- joint link4_Joint: origin xyz=-0.10999 0.01025 0 rpy=0 0 0 -> xyz=-0.109992581095629 0.0102500000277369 0 rpy=0 0 0

Commit message: release: dual-arch (x86_64 + aarch64) 20260609_222116

File: src/human_data/urdf/nexus-arm-v15-right.urdf (robot description, URDF)
Before this commit: robot nexus-arm-v15-right, 9 links, 8 joints
Links:
- link gripper_Link: mass 0.0203179850333118 -> 0.015
- link link1_Link: mass 0.11105324566573 -> 0.1
- link link2_Link: mass 0.817693429898626 -> 0.8
- link link3_Link: mass 0.271751634815028 -> 0.29
- link link4_Link: mass 0.283402825354015 -> 0.33
- link link5_Link: mass 0.313095250711416 -> 0.37
- link link6_Link: mass 0.346716592638755 -> 0.315

Commit message: release: dual-arch (x86_64 + aarch64) 20260611_150724

File: src/human_data/urdf/nexus-arm-v15-right.urdf (robot description, URDF)
Before this commit: robot nexus-arm-v15-right, 9 links, 8 joints
Links:
- link gripper_Link: mass 0.015 -> 0.0203179850333118
- link link1_Link: mass 0.1 -> 0.11105324566573
- link link2_Link: mass 0.8 -> 0.817693429898626
- link link3_Link: mass 0.29 -> 0.271751634815028
- link link4_Link: mass 0.33 -> 0.283402825354015
- link link5_Link: mass 0.37 -> 0.313095250711416
- link link6_Link: mass 0.315 -> 0.346716592638755

File: src/robot_controller/urdf/nexus-arm-v15-right.urdf (robot description, URDF)
Before this commit: robot nexus-arm-v15-right, 9 links, 8 joints
Links:
- link gripper_Link: mass 0.015 -> 0.0203179850333118
- link link1_Link: mass 0.1 -> 0.11105324566573
- link link2_Link: mass 0.8 -> 0.817693429898626
- link link3_Link: mass 0.29 -> 0.271751634815028
- link link4_Link: mass 0.33 -> 0.283402825354015
- link link5_Link: mass 0.37 -> 0.313095250711416
- link link6_Link: mass 0.315 -> 0.346716592638755
Joints:
- joint force_Joint: origin xyz=0 0.08 0 rpy=0 0 0 -> xyz=0 0 0 rpy=0 0 0
