Commit message: release: dual-arch (x86_64 + aarch64) 20260610_202607

File: src/robot_controller/urdf/nexus-arm-v15-right.urdf (robot description, URDF)
Before this commit: robot nexus-arm-v15-right, 9 links, 8 joints
Joints:
- joint force_Joint: origin xyz=0 0 0 rpy=0 0 0 -> xyz=0 0.08 0 rpy=0 0 0

Commit message: release: dual-arch (x86_64 + aarch64) 20260616_155727

File: src/robot_controller/urdf/nexus-arm-v15-right.urdf (robot description, URDF)
Before this commit: robot nexus-arm-v15-right, 9 links, 8 joints
Links:
- link gripper_Link: mass 0.0203179850333118 -> 0.015
- link link1_Link: mass 0.11105324566573 -> 0.1
- link link2_Link: mass 0.817693429898626 -> 0.8
- link link3_Link: mass 0.271751634815028 -> 0.29
- link link4_Link: mass 0.283402825354015 -> 0.33
- link link5_Link: mass 0.313095250711416 -> 0.37
- link link6_Link: mass 0.346716592638755 -> 0.315
Joints:
- joint force_Joint: origin xyz=0 0 0 rpy=0 0 0 -> xyz=0 0.08 0 rpy=0 0 0
